Commit message: added PauseGazebo function, updated packages for gazebo

File: robotics/Ros/src/ur_simulation_gz/ur_simulation_gz/urdf/ur_gz.urdf.xacro (robot description, xacro)
@@ -41,5 +41,5 @@
   </link>
   <joint name="ground_plane_joint" type="fixed">
-    <origin xyz="0 0 -0.01" rpy="0 0 0"/>
+    <origin xyz="0 0 -0.1" rpy="0 0 0"/>
     <parent link="world"/>
     <child link="ground_plane"/>
@@ -59,5 +59,5 @@
     force_abs_paths="true"
     >
-    <origin xyz="0 0 0" rpy="0 0 0" />          <!-- position robot in the world -->
+    <origin xyz="0 0 1.0" rpy="0 0 0" />          <!-- position robot in the world -->
   </xacro:ur_robot>
   <gazebo reference="world">
